File: LoRaDongle.sch (KiCad schematic (older format))
At the start: 31 parts

Commit message: added regulators
Parts:
- removed C?: 470nF, symbol Device:C
- removed C? (x17): C, symbol Device:C
- removed FB?: BLM18AG601SN1D, digikey-footprints:0603, symbol dk_Ferrite-Beads-and-Chips:BLM18AG601SN1D
- removed J?: 142-0701-801, digikey-footprints:RF_SMA_BoardEdge_142-0701-801, symbol dk_Coaxial-Connectors-RF:142-0701-801
- removed L?: 15uH, symbol Device:L
- removed L? (x6): L, symbol Device:L
- removed R?: R, symbol Device:R
- removed U?: SX1262IMLTRT, Semtech-QFN24-0-0-*, symbol sx1262:SX1262IMLTRT
- removed U?: 4259-63, digikey-footprints:SOT-363, symbol dk_RF-Switches:4259-63
- removed U?: XC7A100T-CSG324, symbol FPGA_Xilinx_Artix7:XC7A100T-CSG324
- added J?: USB_A, symbol Connector:USB_A
Connections:
- net labels added: +5V
- net labels removed: !SS, +3V3, DCC_SW, DIO1, DIO2, DIO3, MISO, MOSI, RF1, RFI_N, RFI_P, SCK, VR_PA
- wire segments 95 -> 5
Other:
- note removed: "TODO"

Commit message: updated circuitry
Parts:
- J?: footprint (none) -> Connector_USB:USB_A_CNCTech_1001-011-01101_Horizontal
Changed lines of the file:
@@
 $Descr A4 11693 8268
 encoding utf-8
-Sheet 1 3
+Sheet 1 5
 Title "LoRa Dongle"
 Date ""
@@
 F 0 "J?" H 1057 3567 50  0000 C CNN
 F 1 "USB_A" H 1057 3476 50  0000 C CNN
-F 2 "" H 1150 3050 50  0001 C CNN
+F 2 "Connector_USB:USB_A_CNCTech_1001-011-01101_Horizontal" H 1150 3050 50  0001 C CNN
 F 3 " ~" H 1150 3050 50  0001 C CNN
 	1    1000 3100
@@
 $EndSheet
 $Sheet
-S 8200 3150 1450 800
+S 8000 3000 1450 800
 U 6141DFDA
 F0 "Power Management" 50
 F1 "power_management.sch" 50
 $EndSheet
+$Sheet
+S 7850 4400 1250 700
+U 6149E236
+F0 "fpga_power" 50
+F1 "fpga_power.sch" 50
+$EndSheet
+$Sheet
+S 4400 6450 850  600
+U 618D30E5
+F0 "fpga_configuration" 50
+F1 "fpga_configurarion.sch" 50
+$EndSheet
 $EndSCHEMATC
