File: power_management.sch (KiCad schematic (older format))
At the start: 15 parts

Commit message: updated circuitry
Connections:
- net 3v3 renamed 3V3
Changed lines of the file:
@@
 $Descr A4 11693 8268
 encoding utf-8
-Sheet 3 3
+Sheet 3 5
 Title "LoRa Dongle"
 Date ""
@@
 	4700 2050 4500 2050
 Text GLabel 3400 2050 0    50   Input ~ 0
-3v3
+3V3
 $Comp
 L Device:R R?
