File: LoRaDongle_iCE40_USB/LoRaDongle_iCE40.kicad_sch (KiCad schematic)
At the start: 18 parts, among them J1 USB_A, J2 Conn_01x08, J4 Jumper

Commit message: updating unconnected traces
Connections:
- net USB_Interface/UBS_D+ renamed USB_Interface/USB_D+
Other:
- sheet USB_Interface ports: added USB_D+; removed UBS_D+
Changed lines of the file:
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@@
       (effects (font (size 1.27 1.27)) (justify left))
     )
-    (pin "UBS_D+" input (at 58.42 97.79 180)
+    (pin "USB_D+" input (at 58.42 97.79 180)
       (effects (font (size 1.27 1.27)) (justify left))
     )

Commit message: updating symbol details
Parts:
- 5V0, BUSY1, CDNE1, CRST1, DIO1, L_SS1, MISO1, MOSI1, RESET1, SCK1, SS_B1: Manufacturer (none) -> -; Manufacturer Part Number (none) -> -; Package (none) -> -; Type (none) -> -
- C1: Manufacturer (none) -> Murata Electronics; Manufacturer Part Number (none) -> GCM155R71C104KA55J; Package (none) -> 0402; Type (none) -> SMD
- FB1: Manufacturer Part Number (none) -> BLM18AG601SN1D; Package (none) -> 0603; Type (none) -> SMD
- J1: Manufacturer (none) -> Adam Tech; Manufacturer Part Number (none) -> USB-AP-S-RA-SMT; Package (none) -> Plug; Type (none) -> SMD - Through Hole
- J2, J4: Manufacturer (none) -> -; Manufacturer Part Number (none) -> -; Package (none) -> -; Type (none) -> Through Hole

Commit message: updated BOM
Parts:
- R1, R2: Manufacturer (none) -> Stackpole Electronics Inc; Manufacturer Part Number (none) -> RMCF0402FT10R0; Package (none) -> 0402
Changed lines of the file:
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@@
+      (effects (font (size 1.27 1.27)) hide)
+    )
+    (property "Description" "RES 10 OHM 1% 1/16W 0402" (id 4) (at 50.8 97.79 0)
+      (effects (font (size 1.27 1.27)) hide)
+    )
+    (property "Manufacturer" "Stackpole Electronics Inc" (id 5) (at 50.8 97.79 0)
+      (effects (font (size 1.27 1.27)) hide)
+    )
+    (property "Manufacturer Part Number" "RMCF0402FT10R0" (id 6) (at 50.8 97.79 0)
+      (effects (font (size 1.27 1.27)) hide)
+    )
+    (property "Package" "0402" (id 7) (at 50.8 97.79 0)
       (effects (font (size 1.27 1.27)) hide)
     )
@@
     )
     (property "Datasheet" "~" (id 3) (at 50.8 100.33 0)
+      (effects (font (size 1.27 1.27)) hide)
+    )
+    (property "Description" "RES 10 OHM 1% 1/16W 0402" (id 4) (at 50.8 100.33 0)
+      (effects (font (size 1.27 1.27)) hide)
+    )
+    (property "Manufacturer" "Stackpole Electronics Inc" (id 5) (at 50.8 100.33 0)
+      (effects (font (size 1.27 1.27)) hide)
+    )
+    (property "Manufacturer Part Number" "RMCF0402FT10R0" (id 6) (at 50.8 100.33 0)
+      (effects (font (size 1.27 1.27)) hide)
+    )
+    (property "Package" "0402" (id 7) (at 50.8 100.33 0)
       (effects (font (size 1.27 1.27)) hide)
     )
@@
     )
     (path "/00000000-0000-0000-0000-00006141dfda/00000000-0000-0000-0000-0000616fd330"
-      (reference "D1") (unit 1) (value "LED") (footprint "LED_SMD:LED_0603_1608Metric_Pad1.05x0.95mm_HandSolder")
+      (reference "D1") (unit 1) (value "PWR") (footprint "LED_SMD:LED_0805_2012Metric_Pad1.15x1.40mm_HandSolder")
     )
     (path "/00000000-0000-0000-0000-0000618d30e5/00000000-0000-0000-0000-000061b4f285"
@@
     )
     (path "/00000000-0000-0000-0000-00006141dfda/00000000-0000-0000-0000-0000616fd32a"
-      (reference "R3") (unit 1) (value "R") (footprint "Resistor_SMD:R_0402_1005Metric_Pad0.72x0.64mm_HandSolder")
+      (reference "R3") (unit 1) (value "100R") (footprint "Resistor_SMD:R_0402_1005Metric_Pad0.72x0.64mm_HandSolder")
     )
     (path "/00000000-0000-0000-0000-00006141dfda/00000000-0000-0000-0000-000061449bff"
-      (reference "R4") (unit 1) (value "450K") (footprint "Resistor_SMD:R_0402_1005Metric_Pad0.72x0.64mm_HandSolder")
+      (reference "R4") (unit 1) (value "453K") (footprint "Resistor_SMD:R_0402_1005Metric_Pad0.72x0.64mm_HandSolder")
     )
     (path "/00000000-0000-0000-0000-00006141dfda/00000000-0000-0000-0000-00006144a683"
@@
     )
     (path "/00000000-0000-0000-0000-0000614f0720/00000000-0000-0000-0000-000061687a29"
-      (reference "R20") (unit 1) (value "R") (footprint "Resistor_SMD:R_0402_1005Metric_Pad0.72x0.64mm_HandSolder")
+      (reference "R20") (unit 1) (value "100R") (footprint "Resistor_SMD:R_0402_1005Metric_Pad0.72x0.64mm_HandSolder")
     )
     (path "/00000000-0000-0000-0000-0000614f0720/00000000-0000-0000-0000-00006168ccfd"
-      (reference "R21") (unit 1) (value "R") (footprint "Resistor_SMD:R_0402_1005Metric_Pad0.72x0.64mm_HandSolder")
+      (reference "R21") (unit 1) (value "100R") (footprint "Resistor_SMD:R_0402_1005Metric_Pad0.72x0.64mm_HandSolder")
     )
     (path "/00000000-0000-0000-0000-000061d57b0f"

Commit message: updating silkscreen
Other:
- title: LoRa Dongle -> RiscVLoRaDongle
Changed lines of the file:
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@@
   (paper "A4")
   (title_block
-    (title "LoRa Dongle")
+    (title "RiscVLoRaDongle")
+    (date "2022-02-03")
+    (rev "1.0")
     (company "Mark Njoroge")
   )
+  (junction (at 30.48 110.49) (diameter 0) (color 0 0 0 0)
+  )
   (junction (at 163.83 46.99) (diameter 0) (color 0 0 0 0)
   )
@@
   )
   (junction (at 176.53 102.87) (diameter 0) (color 0 0 0 0)
+  )
+  (junction (at 39.37 92.71) (diameter 0) (color 0 0 0 0)
   )
   (junction (at 163.83 41.91) (diameter 0) (color 0 0 0 0)
@@
     (stroke (width 0) (type default) (color 0 0 0 0))
   )
+  (wire (pts (xy 39.37 92.71) (xy 41.91 92.71))
+    (stroke (width 0) (type default) (color 0 0 0 0))
+  )
   (wire (pts (xy 38.1 97.79) (xy 46.99 97.79))
     (stroke (width 0) (type default) (color 0 0 0 0))
@@
     (stroke (width 0) (type default) (color 0 0 0 0))
   )
+  (wire (pts (xy 30.48 110.49) (xy 30.48 113.03))
+    (stroke (width 0) (type default) (color 0 0 0 0))
+  )
   (wire (pts (xy 161.29 57.15) (xy 171.45 57.15))
     (stroke (width 0) (type default) (color 0 0 0 0))
@@
     (stroke (width 0) (type default) (color 0 0 0 0))
   )
-  (wire (pts (xy 30.48 107.95) (xy 30.48 113.03))
+  (wire (pts (xy 30.48 107.95) (xy 30.48 110.49))
     (stroke (width 0) (type default) (color 0 0 0 0))
   )
@@
     (stroke (width 0) (type default) (color 0 0 0 0))
   )
-  (wire (pts (xy 38.1 92.71) (xy 41.91 92.71))
+  (wire (pts (xy 38.1 92.71) (xy 39.37 92.71))
     (stroke (width 0) (type default) (color 0 0 0 0))
   )
@@
     (pin "1")
   )
+  (symbol (lib_id "power:PWR_FLAG") (at 39.37 92.71 0) (unit 1)
+    (in_bom yes) (on_board yes)
+    (property "Reference" "#FLG02" (id 0) (at 39.37 90.805 0)
+      (effects (font (size 1.27 1.27)) hide)
+    )
+    (property "Value" "PWR_FLAG" (id 1) (at 40.64 88.9 0))
+    (property "Footprint" "" (id 2) (at 39.37 92.71 0)
+      (effects (font (size 1.27 1.27)) hide)
+    )
+    (property "Datasheet" "~" (id 3) (at 39.37 92.71 0)
+      (effects (font (size 1.27 1.27)) hide)
+    )
+    (pin "1")
+  )
+  (symbol (lib_id "power:PWR_FLAG") (at 30.48 110.49 270) (unit 1)
+    (in_bom yes) (on_board yes) (fields_autoplaced)
+    (property "Reference" "#FLG01" (id 0) (at 32.385 110.49 0)
+      (effects (font (size 1.27 1.27)) hide)
+    )
+    (property "Value" "PWR_FLAG" (id 1) (at 34.29 110.4899 90)
+      (effects (font (size 1.27 1.27)) (justify left))
+    )
+    (property "Footprint" "" (id 2) (at 30.48 110.49 0)
+      (effects (font (size 1.27 1.27)) hide)
+    )
+    (property "Datasheet" "~" (id 3) (at 30.48 110.49 0)
+      (effects (font (size 1.27 1.27)) hide)
+    )
+    (pin "1")
+  )
   (sheet (at 67.31 129.54) (size 34.29 19.05) (fields_autoplaced)
     (stroke (width 0) (type solid) (color 0 0 0 0))
@@
   )
   (symbol_instances
+    (path "/bc822dac-2b2d-416d-bac5-21de8ad2c2b0"
+      (reference "#FLG01") (unit 1) (value "PWR_FLAG") (footprint "")
+    )
+    (path "/b177e9c4-328a-40f1-9309-2fbc1f78c015"
+      (reference "#FLG02") (unit 1) (value "PWR_FLAG") (footprint "")
+    )
+    (path "/00000000-0000-0000-0000-00006141dfda/5fc14787-00c1-403d-ae25-801b28391c6c"
+      (reference "#FLG03") (unit 1) (value "PWR_FLAG") (footprint "")
+    )
+    (path "/00000000-0000-0000-0000-0000614f0720/6cf78b91-d5f9-4fff-ad7d-23a13fcd0842"
+      (reference "#FLG04") (unit 1) (value "PWR_FLAG") (footprint "")
+    )
+    (path "/00000000-0000-0000-0000-0000618aacd4/5e60c7b1-29da-4b0f-a8a5-9d1dde438b7e"
+      (reference "#FLG05") (unit 1) (value "PWR_FLAG") (footprint "")
+    )
+    (path "/00000000-0000-0000-0000-0000618aacd4/34951536-903f-41fa-a4c6-c0b93e0bce77"
+      (reference "#FLG06") (unit 1) (value "PWR_FLAG") (footprint "")
+    )
+    (path "/00000000-0000-0000-0000-0000618aacd4/d4aba921-533d-478e-9a8b-92ba53673f2e"
+      (reference "#FLG0101") (unit 1) (value "PWR_FLAG") (footprint "")
+    )
     (path "/00000000-0000-0000-0000-000061702a0e"
       (reference "#PWR01") (unit 1) (value "GND") (footprint "")
