File: LoRaDongle_iCE40_USB/LoRaDongle_iCE40.kicad_pcb (KiCad board)
At the start: 4 copper layers, 110 x 45 mm, 137 parts, among them IC1 93LC56BT-I_OT, IC2 ICE40UP5K-UWG30ITR1K, IC3 N25Q032A13ESC40F, J1 USB_A, J10 Jumper_2_Open, J2 Conn_01x08, J3 Conn_02x02_Top_Bottom, J4 Jumper, J5 142-0701-801, J6 Conn_01x06, J7 Jumper_NC_Small, J8 Jumper, J9 Conn_02x02_Top_Bottom, U1 RP550K001A-TR, U2 FT232H, U3 SX1261IMLTRT, U4 SKY13587-378LF, X1 ECS-2520MV-500-BL-TR, Y1 Crystal_GND24_Small, Y2 Crystal_GND24

Commit message: updated submodules for xilinx
Other:
- board text added: "FTDI BREAKOUT CONNECTOR"
- board text removed: "FT232 BREAKOUT CONNECTOR"
Changed lines of the file:
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@@
     (effects (font (size 1 1) (thickness 0.15)) (justify mirror))
   )
-  (gr_text "FT232 BREAKOUT\n  CONNECTOR" (at 142.65 95.25 90) (layer "B.SilkS")
+  (gr_text "FTDI BREAKOUT\n  CONNECTOR" (at 142.65 95.25 90) (layer "B.SilkS")
     (effects (font (size 1 1) (thickness 0.15)) (justify mirror))
   )
