File: PCB/LoRaDongle_iCE40_USB/USB_Interface.kicad_sch (KiCad schematic)
At the start: 31 parts, among them IC1 93LC56BT-I_OT, J7 Conn_01x03_Male, U2 FT2232HL, Y1 Crystal_GND24_Small

Commit message: updated routing
Connections:
- net CS#: now also IC1.5 (CS), J7.3 (Pin_3), R22.2, U2.63 (EECS)
Changed lines of the file:
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@@
     (effects (font (size 1.27 1.27)) (justify left bottom))
   )
-  (label "CS#" (at 126.238 100.33 90)
+  (label "CS#" (at 125.984 100.33 90)
     (effects (font (size 1.27 1.27)) (justify left bottom))
   )
@@
       (effects (font (size 1.27 1.27)) hide)
     )
-    (property "Description" "RES 10K OHM 1% 1/16W 0402" (id 4) (at 129.032 70.866 0)
+    (property "Description" "RES 12K OHM 1% 1/16W 0402" (id 4) (at 129.032 70.866 0)
       (effects (font (size 1.27 1.27)) hide)
     )
@@
   (symbol (lib_id "Device:R") (at 129.032 75.946 270) (mirror x) (unit 1)
     (in_bom yes) (on_board yes)
-    (property "Reference" "R8" (id 0) (at 129.032 78.486 90))
+    (property "Reference" "R8" (id 0) (at 124.46 74.93 90))
     (property "Value" "1K" (id 1) (at 129.032 75.946 90))
     (property "Footprint" "Resistor_SMD:R_0402_1005Metric_Pad0.72x0.64mm_HandSolder" (id 2) (at 129.032 77.724 90)

Commit message: updated silkscreen
Parts:
- J7: Type (none) -> Through Hole
- R10, R11, R22, R23, R8, R9, U2: Type (none) -> SMD
Changed lines of the file:
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@@
+      (effects (font (size 1.27 1.27)) hide)
+    )
+    (property "Type" "SMD" (id 8) (at 129.032 70.866 0)
       (effects (font (size 1.27 1.27)) hide)
     )
@@
       (effects (font (size 1.27 1.27)) hide)
     )
+    (property "Type" "SMD" (id 8) (at 99.822 111.506 0)
+      (effects (font (size 1.27 1.27)) hide)
+    )
     (pin "1")
     (pin "2")
@@
       (effects (font (size 1.27 1.27)) hide)
     )
+    (property "Type" "SMD" (id 8) (at 93.472 97.028 0)
+      (effects (font (size 1.27 1.27)) hide)
+    )
     (pin "1")
     (pin "2")
@@
       (effects (font (size 1.27 1.27)) hide)
     )
+    (property "Type" "SMD" (id 8) (at 129.032 75.946 0)
+      (effects (font (size 1.27 1.27)) hide)
+    )
     (pin "1")
     (pin "2")
@@
       (effects (font (size 1.27 1.27)) hide)
     )
+    (property "Type" "SMD" (id 8) (at 104.648 97.028 0)
+      (effects (font (size 1.27 1.27)) hide)
+    )
     (pin "1")
     (pin "2")
@@
     )
     (property "Package" "0402" (id 7) (at 101.346 97.028 0)
+      (effects (font (size 1.27 1.27)) hide)
+    )
+    (property "Type" "SMD" (id 8) (at 101.346 97.028 0)
       (effects (font (size 1.27 1.27)) hide)
     )
@@
       (effects (font (size 1.27 1.27)) hide)
     )
+    (property "Type" "Through Hole" (id 8) (at 123.444 90.932 0)
+      (effects (font (size 1.27 1.27)) hide)
+    )
     (pin "1")
     (pin "2")
@@
       (effects (font (size 1.27 1.27)) hide)
     )
+    (property "Type" "SMD" (id 8) (at 169.672 86.106 0)
+      (effects (font (size 1.27 1.27)) hide)
+    )
