File: PCB/LoRaDongle_iCE40_USB/power_management.kicad_sch (KiCad schematic)
At the start: 17 parts, among them U1 RP550K001A-TR

Commit message: updated jumpers, connectors and testpoints
Parts:
- D1: footprint LED_SMD:LED_0805_2012Metric_Pad1.15x1.40mm_HandSolder -> LED_SMD:LED_0603_1608Metric; Manufacturer SunLED -> Lite-On Inc.; Manufacturer Part Number XZM2CRK54WA-8 -> LTST-C191KRKT; Package 0805 -> 0603
Changed lines of the file:
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@@
       (effects (font (size 1.27 1.27)) (justify right))
     )
-    (property "Footprint" "LED_SMD:LED_0805_2012Metric_Pad1.15x1.40mm_HandSolder" (id 2) (at 54.61 104.14 0)
+    (property "Footprint" "LED_SMD:LED_0603_1608Metric" (id 2) (at 54.61 104.14 0)
       (effects (font (size 1.27 1.27)) hide)
     )
@@
       (effects (font (size 1.27 1.27)) hide)
     )
-    (property "Description" "LED RED CLEAR CHIP SMD" (id 4) (at 54.61 104.14 0)
+    (property "Description" "LED RED CLEAR SMD" (id 4) (at 54.61 104.14 0)
       (effects (font (size 1.27 1.27)) hide)
     )
-    (property "Manufacturer" "SunLED" (id 5) (at 54.61 104.14 0)
+    (property "Manufacturer" "Lite-On Inc." (id 5) (at 54.61 104.14 0)
       (effects (font (size 1.27 1.27)) hide)
     )
-    (property "Manufacturer Part Number" "XZM2CRK54WA-8" (id 6) (at 54.61 104.14 0)
+    (property "Manufacturer Part Number" "LTST-C191KRKT" (id 6) (at 54.61 104.14 0)
       (effects (font (size 1.27 1.27)) hide)
     )
-    (property "Package" "0805" (id 7) (at 54.61 104.14 0)
+    (property "Package" "0603" (id 7) (at 54.61 104.14 0)
       (effects (font (size 1.27 1.27)) hide)
     )

Commit message: updated layout and routing
Parts:
- 1V2, 3V3, GND2: footprint TestPoint:TestPoint_Pad_D1.0mm -> TestPoint:TestPoint_Pad_D2.5mm
Changed lines of the file:
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@@
       (effects (font (size 1.27 1.27)) hide)
     )
-    (property "Footprint" "TestPoint:TestPoint_Pad_D1.0mm" (id 2) (at 93.98 83.82 0)
+    (property "Footprint" "TestPoint:TestPoint_Pad_D2.5mm" (id 2) (at 93.98 83.82 0)
       (effects (font (size 1.27 1.27)) hide)
     )
@@
       (effects (font (size 1.27 1.27)) hide)
     )
-    (property "Footprint" "TestPoint:TestPoint_Pad_D1.0mm" (id 2) (at 209.55 83.82 0)
+    (property "Footprint" "TestPoint:TestPoint_Pad_D2.5mm" (id 2) (at 209.55 83.82 0)
       (effects (font (size 1.27 1.27)) hide)
     )
@@
       (effects (font (size 1.27 1.27)) hide)
     )
-    (property "Footprint" "TestPoint:TestPoint_Pad_D1.0mm" (id 2) (at 156.21 121.92 0)
+    (property "Footprint" "TestPoint:TestPoint_Pad_D2.5mm" (id 2) (at 156.21 121.92 0)
       (effects (font (size 1.27 1.27)) hide)
     )

Commit message: updated silkscreen
Parts:
- D1, R3, R4, R5, R6, R7: Type (none) -> SMD
Changed lines of the file:
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@@
+      (effects (font (size 1.27 1.27)) hide)
+    )
+    (property "Type" "SMD" (id 8) (at 184.15 95.25 0)
       (effects (font (size 1.27 1.27)) hide)
     )
@@
     )
     (property "Package" "0402" (id 7) (at 184.15 107.95 0)
+      (effects (font (size 1.27 1.27)) hide)
+    )
+    (property "Type" "SMD" (id 8) (at 184.15 107.95 0)
       (effects (font (size 1.27 1.27)) hide)
     )
@@
       (effects (font (size 1.27 1.27)) hide)
     )
+    (property "Type" "SMD" (id 8) (at 118.11 95.25 0)
+      (effects (font (size 1.27 1.27)) hide)
+    )
     (pin "1")
     (pin "2")
@@
     )
     (property "Package" "0402" (id 7) (at 118.11 107.95 0)
+      (effects (font (size 1.27 1.27)) hide)
+    )
+    (property "Type" "SMD" (id 8) (at 118.11 107.95 0)
       (effects (font (size 1.27 1.27)) hide)
     )
@@
       (effects (font (size 1.27 1.27)) hide)
     )
+    (property "Type" "SMD" (id 8) (at 54.61 95.25 0)
+      (effects (font (size 1.27 1.27)) hide)
+    )
     (pin "1")
     (pin "2")
@@
       (effects (font (size 1.27 1.27)) hide)
     )
+    (property "Type" "SMD" (id 8) (at 54.61 104.14 0)
+      (effects (font (size 1.27 1.27)) hide)
+    )
