File: PCB/LoRaDongle_iCE40_USB/sx1261_circuitry.kicad_sch (KiCad schematic)
At the start: 42 parts, among them J5 142-0701-801, J8 Jumper_2_Open, U3 SX1261IMLTRT, U4 SKY13587-378LF, Y2 Crystal_GND24

Commit message: updated routing
Parts:
- J5: Manufacturer Part Number (none) -> 142-0701-801
Changed lines of the file:
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@@
       (effects (font (size 1.524 1.524)) (justify left) hide)
+    )
+    (property "Manufacturer Part Number" "142-0701-801" (id 13) (at 209.55 111.76 0)
+      (effects (font (size 1.27 1.27)) hide)
     )
     (pin "1")

Commit message: updated BOM
Parts:
- J5: Package (none) -> Connector
Changed lines of the file:
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@@
+      (effects (font (size 1.27 1.27)) hide)
+    )
+    (property "Package" "Connector" (id 14) (at 209.55 111.76 0)
       (effects (font (size 1.27 1.27)) hide)
     )

Commit message: updated silkscreen
Parts:
- D3, D4, J5, R18, R19, R20, R21: Type (none) -> SMD
- J8: Type (none) -> Through Hole
- L8: Package (none) -> 0402; Type (none) -> SMD
Changed lines of the file:
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@@
+      (effects (font (size 1.27 1.27)) hide)
+    )
+    (property "Type" "SMD" (id 8) (at 199.39 48.26 0)
+      (effects (font (size 1.27 1.27)) hide)
+    )
+    (property "Package" "0402" (id 9) (at 199.39 48.26 0)
       (effects (font (size 1.27 1.27)) hide)
     )
@@
       (effects (font (size 1.27 1.27)) hide)
     )
+    (property "Type" "SMD" (id 9) (at 130.81 146.05 0)
+      (effects (font (size 1.27 1.27)) hide)
+    )
     (pin "1")
     (pin "2")
@@
       (effects (font (size 1.27 1.27)) hide)
     )
+    (property "Type" "SMD" (id 8) (at 247.65 127 0)
+      (effects (font (size 1.27 1.27)) hide)
+    )
     (pin "1")
     (pin "2")
@@
       (effects (font (size 1.27 1.27)) hide)
     )
+    (property "Type" "SMD" (id 8) (at 247.65 135.89 0)
+      (effects (font (size 1.27 1.27)) hide)
+    )
     (pin "1")
     (pin "2")
@@
       (effects (font (size 1.27 1.27)) hide)
     )
+    (property "Type" "SMD" (id 8) (at 261.62 127 0)
+      (effects (font (size 1.27 1.27)) hide)
+    )
     (pin "1")
     (pin "2")
@@
     )
     (property "Package" "0603" (id 7) (at 261.62 135.89 0)
+      (effects (font (size 1.27 1.27)) hide)
+    )
+    (property "Type" "SMD" (id 8) (at 261.62 135.89 0)
       (effects (font (size 1.27 1.27)) hide)
     )
@@
     )
     (property "Package" "0402" (id 8) (at 171.45 146.05 0)
+      (effects (font (size 1.27 1.27)) hide)
+    )
+    (property "Type" "SMD" (id 9) (at 171.45 146.05 0)
       (effects (font (size 1.27 1.27)) hide)
     )
@@
       (effects (font (size 1.27 1.27)) hide)
     )
+    (property "Type" "SMD" (id 15) (at 209.55 111.76 0)
+      (effects (font (size 1.27 1.27)) hide)
+    )
     (pin "1")
     (pin "2")
@@
       (effects (font (size 1.27 1.27)) hide)
     )
+    (property "Type" "Through Hole" (id 8) (at 35.56 92.71 0)
+      (effects (font (size 1.27 1.27)) hide)
+    )
